File: hardware/eagle/nixie_clock.sch (EAGLE design)
At the start: 39 parts, among them IC1 74141N, IC10 74141N, IC11 7477N, IC12 74141N, IC13 7477N, IC14 74AC11238, IC2 7477N, IC4 74141N, IC5 7477N, IC6 74141N, IC7 7477N, IC8 74141N, IC9 7477N

Commit message: First board
Parts:
- removed IC14: 74AC11238, 74ac-logic:74AC11238
- added IC3: 74141N, 74xx-eu:74141N
- added J1_180V, J1_180V1: 22-27-2021-02, con-molex:22-27-2021-02
- IC10, IC12, IC4, IC6, IC8: value 74141N -> 7477N; device 74xx-eu:74141N -> 74xx-eu:7477N
- IC11, IC5, IC7, IC9: value 7477N -> 74141N; device 74xx-eu:7477N -> 74xx-eu:74141N
- IC13: value 7477N -> 74AC11238; device 74xx-eu:7477N -> 74ac-logic:74AC11238
Connections:
- net +5V: now also IC13A.G1, IC3P.VCC, J1_180V1-1.S; no longer IC14A.G1, IC14P.VCC
- net GND: now also IC13A.G2A, IC13A.G2B, IC3P.GND, J1_180V-1.S, J1_180V1-2.S; no longer IC14A.G2A, IC14A.G2B, IC14P.GND
- net N$1: now also IN-8-1.A; no longer IN-8-2.A
- net N$10: now also IN-8-1.9; no longer IN-8-2.9
- net N$11: now also IN-8-1.0; no longer IN-8-2.0
- net N$16: now also IC13A.Y0; no longer IC14A.Y0
- net N$17: now also IC10A.4D, IC12A.4D, IC4A.4D, IC6A.4D, IC8A.4D; no longer IC11A.4D, IC13A.4D, IC5A.4D, IC7A.4D, IC9A.4D
- net N$18: now also IN-8-2.A; no longer IN-8-1.A
- net N$19: now also IC3A.1, IN-8-2.1; no longer IC4A.1, IN-8-1.1
- net N$2: now also IN-8-1.1; no longer IN-8-2.1
- net N$20: now also IC3A.2, IN-8-2.2; no longer IC4A.2, IN-8-1.2
- net N$21: now also IC3A.3, IN-8-2.3; no longer IC4A.3, IN-8-1.3
- net N$22: now also IC3A.4, IN-8-2.4; no longer IC4A.4, IN-8-1.4
- net N$23: now also IC3A.5, IN-8-2.5; no longer IC4A.5, IN-8-1.5
- net N$24: now also IC3A.6, IN-8-2.6; no longer IC4A.6, IN-8-1.6
- net N$25: now also IC3A.7, IN-8-2.7; no longer IC4A.7, IN-8-1.7
- net N$26: now also IC3A.8, IN-8-2.8; no longer IC4A.8, IN-8-1.8
- net N$27: now also IC3A.9, IN-8-2.9; no longer IC4A.9, IN-8-1.9
- net N$28: now also IC3A.0, IN-8-2.0; no longer IC4A.0, IN-8-1.0
- net N$29: now also IC3A.A, IC4A.1Q; no longer IC4A.A, IC5A.1Q
- net N$3: now also IN-8-1.2; no longer IN-8-2.2
- net N$30: now also IC3A.B, IC4A.2Q; no longer IC4A.B, IC5A.2Q
- net N$31: now also IC3A.C, IC4A.3Q; no longer IC4A.C, IC5A.3Q
- net N$32: now also IC3A.D, IC4A.4Q; no longer IC4A.D, IC5A.4Q
- net N$33: now also IC13A.Y1, IC4A.12C, IC4A.34C; no longer IC14A.Y1, IC5A.12C, IC5A.34C
- net N$34: now also IC5A.1; no longer IC6A.1
- net N$35: now also IC5A.2; no longer IC6A.2
- net N$36: now also IC5A.3; no longer IC6A.3
- net N$37: now also IC5A.4; no longer IC6A.4
- net N$38: now also IC5A.5; no longer IC6A.5
- net N$39: now also IC5A.6; no longer IC6A.6
- net N$4: now also IN-8-1.3; no longer IN-8-2.3
- net N$40: now also IC5A.7; no longer IC6A.7
- net N$41: now also IC5A.8; no longer IC6A.8
- net N$42: now also IC5A.9; no longer IC6A.9
- net N$43: now also IC5A.0; no longer IC6A.0
- net N$44: now also IC5A.A, IC6A.1Q; no longer IC6A.A, IC7A.1Q
- net N$45: now also IC5A.B, IC6A.2Q; no longer IC6A.B, IC7A.2Q
- net N$46: now also IC5A.C, IC6A.3Q; no longer IC6A.C, IC7A.3Q
- net N$47: now also IC5A.D, IC6A.4Q; no longer IC6A.D, IC7A.4Q
- net N$48: now also IC13A.Y2, IC6A.12C, IC6A.34C; no longer IC14A.Y2, IC7A.12C, IC7A.34C
- net N$49: now also IC7A.1; no longer IC8A.1
- net N$5: now also IN-8-1.4; no longer IN-8-2.4
- net N$50: now also IC7A.2; no longer IC8A.2
- net N$51: now also IC7A.3; no longer IC8A.3
- net N$52: now also IC7A.4; no longer IC8A.4
- net N$53: now also IC7A.5; no longer IC8A.5
- net N$54: now also IC7A.6; no longer IC8A.6
- net N$55: now also IC7A.7; no longer IC8A.7
- net N$56: now also IC7A.8; no longer IC8A.8
- net N$57: now also IC7A.9; no longer IC8A.9
- net N$58: now also IC7A.0; no longer IC8A.0
- net N$59: now also IC7A.A, IC8A.1Q; no longer IC8A.A, IC9A.1Q
- net N$6: now also IN-8-1.5; no longer IN-8-2.5
- net N$60: now also IC7A.B, IC8A.2Q; no longer IC8A.B, IC9A.2Q
- net N$61: now also IC7A.C, IC8A.3Q; no longer IC8A.C, IC9A.3Q
- net N$62: now also IC7A.D, IC8A.4Q; no longer IC8A.D, IC9A.4Q
- net N$63: now also IC13A.Y3, IC8A.12C, IC8A.34C; no longer IC14A.Y3, IC9A.12C, IC9A.34C
- net N$64: now also IC9A.1; no longer IC10A.1
- net N$65: now also IC9A.2; no longer IC10A.2
- net N$66: now also IC9A.3; no longer IC10A.3
- net N$67: now also IC9A.4; no longer IC10A.4
- net N$68: now also IC9A.5; no longer IC10A.5
- net N$69: now also IC9A.6; no longer IC10A.6
- net N$7: now also IN-8-1.6; no longer IN-8-2.6
- net N$70: now also IC9A.7; no longer IC10A.7
- net N$71: now also IC9A.8; no longer IC10A.8
- net N$72: now also IC9A.9; no longer IC10A.9
- net N$73: now also IC9A.0; no longer IC10A.0
- net N$74: now also IC10A.1Q, IC9A.A; no longer IC10A.A, IC11A.1Q
- net N$75: now also IC10A.2Q, IC9A.B; no longer IC10A.B, IC11A.2Q
- net N$76: now also IC10A.3Q, IC9A.C; no longer IC10A.C, IC11A.3Q
- net N$77: now also IC10A.4Q, IC9A.D; no longer IC10A.D, IC11A.4Q
- net N$78: now also IC10A.12C, IC10A.34C, IC13A.Y4; no longer IC11A.12C, IC11A.34C, IC14A.Y4
- net N$79: now also IC11A.1; no longer IC12A.1
- net N$8: now also IN-8-1.7; no longer IN-8-2.7
- net N$80: now also IC11A.2; no longer IC12A.2
- net N$81: now also IC11A.3; no longer IC12A.3
- net N$82: now also IC11A.4; no longer IC12A.4
- net N$83: now also IC11A.5; no longer IC12A.5
- net N$84: now also IC11A.6; no longer IC12A.6
- net N$85: now also IC11A.7; no longer IC12A.7
- net N$86: now also IC11A.8; no longer IC12A.8
- net N$87: now also IC11A.9; no longer IC12A.9
- net N$88: now also IC11A.0; no longer IC12A.0
- net N$89: now also IC11A.A, IC12A.1Q; no longer IC12A.A, IC13A.1Q
- net N$9: now also IN-8-1.8; no longer IN-8-2.8
- net N$90: now also IC11A.B, IC12A.2Q; no longer IC12A.B, IC13A.2Q
- net N$91: now also IC11A.C, IC12A.3Q; no longer IC12A.C, IC13A.3Q
- net N$92: now also IC11A.D, IC12A.4Q; no longer IC12A.D, IC13A.4Q
- net N$93: now also IC12A.12C, IC12A.34C, IC13A.Y5; no longer IC13A.12C, IC13A.34C, IC14A.Y5
- net N$94: now also IC10A.3D, IC12A.3D, IC4A.3D, IC6A.3D, IC8A.3D; no longer IC11A.3D, IC13A.3D, IC5A.3D, IC7A.3D, IC9A.3D
- net N$95: now also IC10A.2D, IC12A.2D, IC4A.2D, IC6A.2D, IC8A.2D; no longer IC11A.2D, IC13A.2D, IC5A.2D, IC7A.2D, IC9A.2D
- net N$96: now also IC10A.1D, IC12A.1D, IC4A.1D, IC6A.1D, IC8A.1D; no longer IC11A.1D, IC13A.1D, IC5A.1D, IC7A.1D, IC9A.1D
- net N$97: now also IC13A.A; no longer IC14A.A
- net N$98: now also IC13A.B; no longer IC14A.B
- net N$99: now also IC13A.C; no longer IC14A.C
- net VCC: now also J1_180V-2.S
Other:
- moved on the sheet: IC10P, IC11P, IC12P, IC13P, IC4P, IC5P, IC6P, IC7P, IC8P, IC9P, IN-8-1, IN-8-2

Commit message: Updated eagle project
Parts:
- removed J1_180V1: 22-27-2021-02, con-molex:22-27-2021-02
- added J1_5V1: 22-27-2021-02, con-molex:22-27-2021-02
- R1, R2, R3, R4, R5, R6: device resistor:R-EU_0204/5 -> resistor:R-EU_0207/15
Connections:
- removed net +5V: C1.2, C10.2, C11.2, C12.2, C13.2, C2.2, C3.2, C4.2, C5.2, C6.2, C7.2, C8.2, C9.2, IC10P.VCC, IC11P.VCC, IC12P.VCC, IC13A.G1, IC13P.VCC, IC1P.VCC, IC2P.VCC, IC3P.VCC, IC4P.VCC, IC5P.VCC, IC6P.VCC, IC7P.VCC, IC8P.VCC, IC9P.VCC, J1_180V1-1.S
- new net N$108: C1.2, C10.2, C11.2, C12.2, C13.2, C2.2, C3.2, C4.2, C5.2, C6.2, C7.2, C8.2, C9.2, IC10P.VCC, IC11P.VCC, IC12P.VCC, IC13A.G1, IC13P.VCC, IC1P.VCC, IC2P.VCC, IC3P.VCC, IC4P.VCC, IC5P.VCC, IC6P.VCC, IC7P.VCC, IC8P.VCC, IC9P.VCC, J1_5V1-2.S
- net GND: now also J1_5V1-1.S; no longer J1_180V1-2.S
Other:
- moved on the sheet: C1, C10, C11, C12, C13, C2, C3, C4, C5, C6, C7, C8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

Commit message: External nixie tubes design
Parts:
- removed IN-8-2, IN-8-3, IN-8-4, IN-8-5, IN-8-6: IN-8-2, russian-nixies:IN-8-2
- added SV1, SV11, SV13, SV3, SV5, SV7, SV9: (no value), con-lstb:MA06-1
- added SV10, SV12, SV14, SV2, SV4, SV6, SV8: (no value), con-lstb:MA05-1
Connections:
- new net N$104: IN-8-1.1, SV14.2
- new net N$105: IN-8-1.2, SV14.3
- new net N$106: IN-8-1.3, SV14.4
- new net N$107: IN-8-1.4, SV14.5
- new net N$109: IN-8-1.5, SV13.1
- new net N$110: IN-8-1.6, SV13.2
- new net N$111: IN-8-1.7, SV13.3
- new net N$112: IN-8-1.8, SV13.4
- new net N$113: IN-8-1.9, SV13.5
- new net N$114: IN-8-1.0, SV14.1
- new net N$115: IN-8-1.A, SV13.6
- net N$1: now also IC3A.5, SV3.1; no longer IN-8-1.A, R1.1
- net N$10: now also IC1A.8, SV1.4; no longer IC1A.9, IN-8-1.9
- net N$100: now also R3.1, SV5.6; no longer IN-8-4.A, R4.1
- net N$101: now also R4.1, SV7.6; no longer IN-8-5.A, R5.1
- net N$102: now also R5.1, SV9.6; no longer IN-8-6.A, R6.1
- net N$103: now also R6.1, SV11.6; no longer IN-8-3.A, R3.1
- net N$11: now also IC1A.9, SV1.5; no longer IC1A.0, IN-8-1.0
- net N$18: now also IC3A.8, SV3.4; no longer IN-8-2.A, R2.1
- net N$19: now also IC3A.0, SV4.1; no longer IC3A.1, IN-8-2.1
- net N$2: now also IC1A.0, SV2.1; no longer IC1A.1, IN-8-1.1
- net N$20: now also IC3A.1, SV4.2; no longer IC3A.2, IN-8-2.2
- net N$21: now also IC3A.2, SV4.3; no longer IC3A.3, IN-8-2.3
- net N$22: now also IC3A.3, SV4.4; no longer IC3A.4, IN-8-2.4
- net N$23: now also IC3A.4, SV4.5; no longer IC3A.5, IN-8-2.5
- net N$24: now also IC7A.5, SV7.1; no longer IC3A.6, IN-8-2.6
- net N$25: now also IC7A.6, SV7.2; no longer IC3A.7, IN-8-2.7
- net N$26: now also IC7A.7, SV7.3; no longer IC3A.8, IN-8-2.8
- net N$27: now also IC7A.8, SV7.4; no longer IC3A.9, IN-8-2.9
- net N$28: now also IC7A.9, SV7.5; no longer IC3A.0, IN-8-2.0
- net N$3: now also IC1A.1, SV2.2; no longer IC1A.2, IN-8-1.2
- net N$34: now also IC5A.0, SV6.1; no longer IC5A.1, IN-8-3.1
- net N$35: now also IC5A.1, SV6.2; no longer IC5A.2, IN-8-3.2
- net N$36: now also IC5A.2, SV6.3; no longer IC5A.3, IN-8-3.3
- net N$37: now also IC5A.3, SV6.4; no longer IC5A.4, IN-8-3.4
- net N$38: now also IC5A.4, SV6.5; no longer IC5A.5, IN-8-3.5
- net N$39: now also IC9A.5, SV9.1; no longer IC5A.6, IN-8-3.6
- net N$4: now also IC1A.2, SV2.3; no longer IC1A.3, IN-8-1.3
- net N$40: now also IC9A.6, SV9.2; no longer IC5A.7, IN-8-3.7
- net N$41: now also IC9A.7, SV9.3; no longer IC5A.8, IN-8-3.8
- net N$42: now also IC9A.8, SV9.4; no longer IC5A.9, IN-8-3.9
- net N$43: now also IC9A.9, SV9.5; no longer IC5A.0, IN-8-3.0
- net N$49: now also IC7A.0, SV8.1; no longer IC7A.1, IN-8-4.1
- net N$5: now also IC1A.3, SV2.4; no longer IC1A.4, IN-8-1.4
- net N$50: now also IC7A.1, SV8.2; no longer IC7A.2, IN-8-4.2
- net N$51: now also IC7A.2, SV8.3; no longer IC7A.3, IN-8-4.3
- net N$52: now also IC7A.3, SV8.4; no longer IC7A.4, IN-8-4.4
- net N$53: now also IC7A.4, SV8.5; no longer IC7A.5, IN-8-4.5
- net N$54: now also IC11A.5, SV11.1; no longer IC7A.6, IN-8-4.6
- net N$55: now also IC11A.6, SV11.2; no longer IC7A.7, IN-8-4.7
- net N$56: now also IC11A.7, SV11.3; no longer IC7A.8, IN-8-4.8
- net N$57: now also IC11A.8, SV11.4; no longer IC7A.9, IN-8-4.9
- net N$58: now also IC11A.9, SV11.5; no longer IC7A.0, IN-8-4.0
- net N$6: now also IC1A.4, SV2.5; no longer IC1A.5, IN-8-1.5
- net N$64: now also IC9A.0, SV10.1; no longer IC9A.1, IN-8-5.1
- net N$65: now also IC9A.1, SV10.2; no longer IC9A.2, IN-8-5.2
- net N$66: now also IC9A.2, SV10.3; no longer IC9A.3, IN-8-5.3
- net N$67: now also IC9A.3, SV10.4; no longer IC9A.4, IN-8-5.4
- net N$68: now also IC9A.4, SV10.5; no longer IC9A.5, IN-8-5.5
- net N$69: now also IC3A.6, SV3.2; no longer IC9A.6, IN-8-5.6
- net N$7: now also IC1A.5, SV1.1; no longer IC1A.6, IN-8-1.6
- net N$70: now also IC3A.7, SV3.3; no longer IC9A.7, IN-8-5.7
- net N$71: now also IC3A.9, SV3.5; no longer IC9A.8, IN-8-5.8
- net N$72: now also R2.1, SV3.6; no longer IC9A.9, IN-8-5.9
- net N$73: now also R1.1, SV1.6; no longer IC9A.0, IN-8-5.0
- net N$79: now also IC11A.0, SV12.1; no longer IC11A.1, IN-8-6.1
- net N$8: now also IC1A.6, SV1.2; no longer IC1A.7, IN-8-1.7
- net N$80: now also IC11A.1, SV12.2; no longer IC11A.2, IN-8-6.2
- net N$81: now also IC11A.2, SV12.3; no longer IC11A.3, IN-8-6.3
- net N$82: now also IC11A.3, SV12.4; no longer IC11A.4, IN-8-6.4
- net N$83: now also IC11A.4, SV12.5; no longer IC11A.5, IN-8-6.5
- net N$84: now also IC5A.5, SV5.1; no longer IC11A.6, IN-8-6.6
- net N$85: now also IC5A.6, SV5.2; no longer IC11A.7, IN-8-6.7
- net N$86: now also IC5A.7, SV5.3; no longer IC11A.8, IN-8-6.8
- net N$87: now also IC5A.8, SV5.4; no longer IC11A.9, IN-8-6.9
- net N$88: now also IC5A.9, SV5.5; no longer IC11A.0, IN-8-6.0
- net N$9: now also IC1A.7, SV1.3; no longer IC1A.8, IN-8-1.8
Other:
- moved on the sheet: IN-8-1, J1_180V-1, J1_180V-2, R1, R2, R3, R4, R5, R6

Commit message: Updated eagle project
Connections:
- removed net N$105 (its old number): IN-8-1.2, SV14.3
- removed net N$19 (its old number): IC3A.0, SV4.1
- removed net N$2 (its old number): IC1A.0, SV2.1
- removed net N$4 (its old number): IC1A.2, SV2.3
- removed net N$5 (its old number): IC1A.3, SV2.4
- removed net N$51 (its old number): IC7A.2, SV8.3
- removed net N$67 (its old number): IC9A.3, SV10.4
- removed net N$7 (its old number): IC1A.5, SV1.1
- removed net N$84 (its old number): IC5A.5, SV5.1
- new net N$104: IN-8-1.A, SV14.3
- new net N$12: IC1A.4, SV1.2
- new net N$13: IC1A.5, SV1.3
- new net N$14: IC1A.6, SV1.4
- new net N$15: IC1A.7, SV1.5
- new net N$20: IC3A.0, SV4.4
- new net N$50: IC7A.2, SV8.1
- new net N$65: R5.1, SV10.3
- new net N$80: IC9A.7, SV9.5
- net N$1: now also R2.1, SV4.3; no longer IC3A.5, SV3.1
- net N$10: now also IC1A.9, SV2.5; no longer IC1A.8, SV1.4
- net N$100: now also IC11A.5, SV11.3; no longer R3.1, SV5.6
- net N$101: now also IC11A.6, SV11.4; no longer R4.1, SV7.6
- net N$102: now also IC11A.7, SV11.5; no longer R5.1, SV9.6
- net N$103: now also IC11A.8; no longer R6.1
- net N$106: now also IN-8-1.2, SV14.1; no longer IN-8-1.3, SV14.4
- net N$107: now also IN-8-1.0, SV14.4; no longer IN-8-1.4, SV14.5
- net N$109: now also IN-8-1.9, SV14.5; no longer IN-8-1.5, SV13.1
- net N$11: now also IC1A.3, SV1.1; no longer IC1A.9, SV1.5
- net N$110: now also IN-8-1.8, SV13.6; no longer IN-8-1.6, SV13.2
- net N$111: now also SV13.5; no longer SV13.3
- net N$112: now also IN-8-1.6; no longer IN-8-1.8
- net N$113: now also IN-8-1.5, SV13.3; no longer IN-8-1.9, SV13.5
- net N$114: now also IN-8-1.4, SV13.2; no longer IN-8-1.0, SV14.1
- net N$115: now also IN-8-1.3, SV13.1; no longer IN-8-1.A, SV13.6
- net N$18: now also IC3A.2, SV4.1; no longer IC3A.8, SV3.4
- net N$21: now also IC3A.9, SV4.5; no longer IC3A.2, SV4.3
- net N$22: now also SV3.1; no longer SV4.4
- net N$23: now also SV3.2; no longer SV4.5
- net N$24: now also IC3A.5, SV3.3; no longer IC7A.5, SV7.1
- net N$25: now also IC3A.6, SV3.4; no longer IC7A.6, SV7.2
- net N$26: now also IC3A.7, SV3.5; no longer IC7A.7, SV7.3
- net N$27: now also IC3A.8, SV3.6; no longer IC7A.8, SV7.4
- net N$28: now also R3.1, SV6.3; no longer IC7A.9, SV7.5
- net N$34: now also IC5A.2; no longer IC5A.0
- net N$36: now also IC5A.0, SV6.4; no longer IC5A.2, SV6.3
- net N$37: now also IC5A.9, SV6.5; no longer IC5A.3, SV6.4
- net N$38: now also IC5A.3, SV5.1; no longer IC5A.4, SV6.5
- net N$39: now also IC5A.4, SV5.2; no longer IC9A.5, SV9.1
- net N$40: now also IC5A.5, SV5.3; no longer IC9A.6, SV9.2
- net N$41: now also IC5A.6, SV5.4; no longer IC9A.7, SV9.3
- net N$42: now also IC5A.7, SV5.5; no longer IC9A.8, SV9.4
- net N$43: now also IC5A.8, SV5.6; no longer IC9A.9, SV9.5
- net N$49: now also R4.1, SV8.3; no longer IC7A.0, SV8.1
- net N$52: now also IC7A.0; no longer IC7A.3
- net N$53: now also IC7A.9; no longer IC7A.4
- net N$54: now also IC7A.3, SV7.1; no longer IC11A.5, SV11.1
- net N$55: now also IC7A.4, SV7.2; no longer IC11A.6, SV11.2
- net N$56: now also IC7A.5, SV7.3; no longer IC11A.7, SV11.3
- net N$57: now also IC7A.6, SV7.4; no longer IC11A.8, SV11.4
- net N$58: now also IC7A.7, SV7.5; no longer IC11A.9, SV11.5
- net N$6: now also R1.1, SV2.3; no longer IC1A.4, SV2.5
- net N$64: now also IC7A.8, SV7.6; no longer IC9A.0, SV10.1
- net N$66: now also SV10.1; no longer SV10.3
- net N$68: now also IC9A.0, SV10.4; no longer IC9A.4, SV10.5
- net N$69: now also IC9A.9, SV10.5; no longer IC3A.6, SV3.2
- net N$70: now also IC9A.3, SV9.1; no longer IC3A.7, SV3.3
- net N$71: now also IC9A.4, SV9.2; no longer IC3A.9, SV3.5
- net N$72: now also IC9A.5, SV9.3; no longer R2.1, SV3.6
- net N$73: now also IC1A.8; no longer R1.1
- net N$79: now also IC9A.6, SV9.4; no longer IC11A.0, SV12.1
- net N$8: now also IC1A.2, SV2.1; no longer IC1A.6, SV1.2
- net N$81: now also IC9A.8, SV9.6; no longer IC11A.2, SV12.3
- net N$82: now also R6.1, SV12.3; no longer IC11A.3, SV12.4
- net N$83: now also IC11A.2, SV12.1; no longer IC11A.4, SV12.5
- net N$85: now also IC11A.0, SV12.4; no longer IC5A.6, SV5.2
- net N$86: now also IC11A.9, SV12.5; no longer IC5A.7, SV5.3
- net N$87: now also IC11A.3, SV11.1; no longer IC5A.8, SV5.4
- net N$88: now also IC11A.4, SV11.2; no longer IC5A.9, SV5.5
- net N$9: now also IC1A.0, SV2.4; no longer IC1A.7, SV1.3
Other:
- moved on the sheet: SV1, SV10, SV11, SV12, SV2, SV3, SV4, SV5, SV6, SV7, SV8, SV9

Commit message: Added power supply on eagle project
Parts:
- added B1: (no value), rectifier:FBP1,5
- added C14: (no value), rcl:CPOL-EUE5-10.5
- added C15: (no value), rcl:CPOL-EUE3.5-10
- added F1, F2: FUSESH22,5A, fuse:FUSESH22,5A
- added IC14: (no value), v-reg:78XXS
- added J1_5V2: 22-27-2021-02, con-molex:22-27-2021-02
- added KK1: FK218, heatsink:FK218
- added LSP1, LSP2: LSP10, solpad:LSP10
- added TR1: (no value), trafo:EI42-1
Connections:
- new net N$108: B1.+, C14.+, IC14.IN
- new net N$117: F1.1, LSP1.MP
- new net N$118: F1.2, TR1.P1
- new net N$119: LSP2.MP, TR1.P2
- new net N$120: F2.1, TR1.S4
- new net N$121: B1.AC1, F2.2
- new net N$122: B1.AC2, TR1.S3
- new net N$123: C15.+, IC14.OUT, J1_5V2-2.S
- new net N$125: B1.-, C14.-, C15.-, IC14.GND, J1_5V2-1.S
Other:
- moved on the sheet: J1_5V1-1, J1_5V1-2, SV13, SV14
