File: hardware/eagle/nixie_clock.sch (EAGLE design)
At the start: 84 parts, among them IC1 74141N, IC10 7477N, IC11 74141N, IC12 7477N, IC13 74HCT259N, IC15 7477N, IC2 7477N, IC3 74141N, IC4 7477N, IC5 74141N, IC6 7477N, IC7 74141N, IC8 7477N, IC9 74141N, J1 RASPBERRYPI-40-PIN-GPIO, J1_180V 22-27-2021-02, J1_5V1 22-27-2021-02, J1_5V2 22-27-2021-02, K1 4052, SW1 ROTARTY_ENCODER

Commit message: Updated eagle project
Parts:
- added J11: (no value), SparkFun-Connectors:M03PTH
- SV15, SV16: device con-lstb:MA05-1 -> SparkFun-Connectors:M05PTH
Connections:
- removed net GROUND: C1.2, C10.2, C11.2, C12.2, C13.2, C16.2, C17.2, C2.2, C3.2, C4.2, C5.2, C6.2, C7.2, C8.2, C9.2, D2.A, IC10P.VCC, IC11P.VCC, IC12P.VCC, IC13A.D, IC13P.VCC, IC15P.VCC, IC1P.VCC, IC2P.VCC, IC3P.VCC, IC4P.VCC, IC5P.VCC, IC6P.VCC, IC7P.VCC, IC8P.VCC, IC9P.VCC, J1_5V1-2.S, J3.4, K11.2, R12.2, R7.2, R8.1, SV10.5, SV12.5, SV16.1, SV2.5, SV4.5, SV6.5, SV8.5, ULN1.10
- new net 5V: C1.2, C10.2, C11.2, C12.2, C13.2, C16.2, C17.2, C2.2, C3.2, C4.2, C5.2, C6.2, C7.2, C8.2, C9.2, D2.A, IC10P.VCC, IC11P.VCC, IC12P.VCC, IC13A.D, IC13P.VCC, IC15P.VCC, IC1P.VCC, IC2P.VCC, IC3P.VCC, IC4P.VCC, IC5P.VCC, IC6P.VCC, IC7P.VCC, IC8P.VCC, IC9P.VCC, J11.2, J1_5V1-2.S, J3.4, K11.2, R12.2, R7.2, R8.1, SV10.5, SV12.5, SV16.1, SV2.5, SV4.5, SV6.5, SV8.5, ULN1.10
- new net N$173: J1.GP16, J11.3
- net GND: now also J11.1
Other:
- note added: "3.3V"
- note added: "5V"
- note added: "CE0"
- note added: "CE1"
- note added: "ID_SC"
- note added: "ID_SD"
- note added: "MISO"
- note added: "MOSI"
- note added: "PIR_OUT"
- note added: "RX"
- note added: "SCL"
- note added: "SCLK"
- note added: "SDA"
- note added: "TX"
- moved on the sheet: SV15, SV16, SW1
Changed lines of the file:
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@@
 <part name="D2" library="diode" deviceset="1N4004" device=""/>
 <part name="SW1" library="SparkFun-Electromechanical" deviceset="ROTARTY_ENCODER" device=""/>
-<part name="SV15" library="con-lstb" deviceset="MA05-1" device=""/>
-<part name="SV16" library="con-lstb" deviceset="MA05-1" device=""/>
+<part name="SV15" library="SparkFun-Connectors" deviceset="M05" device="PTH"/>
+<part name="SV16" library="SparkFun-Connectors" deviceset="M05" device="PTH"/>
 <part name="ULN1" library="SparkFun-PowerIC" deviceset="ULN2803" device="DIP"/>
 <part name="D1" library="SparkFun-LED" deviceset="LED-RGB-CA-THRU" device="CLEAR"/>
@@
 <part name="J9" library="SparkFun-Connectors" deviceset="M08" device=""/>
 <part name="J10" library="SparkFun-Connectors" deviceset="M08" device=""/>
+<part name="J11" library="SparkFun-Connectors" deviceset="M03" device="PTH"/>
 </parts>
 <sheets>
@@
 <text x="299.72" y="96.52" size="1.778" layer="95">GND</text>
 <text x="299.72" y="99.06" size="1.778" layer="95">VCC</text>
+<text x="327.66" y="215.9" size="1.778" layer="95">3.3V</text>
+<text x="327.66" y="190.5" size="1.778" layer="95">3.3V</text>
+<text x="327.66" y="187.96" size="1.778" layer="95">SDA</text>
+<text x="327.66" y="185.42" size="1.778" layer="95">SCL</text>
+<text x="327.66" y="182.88" size="1.778" layer="95">ID_SD</text>
+<text x="327.66" y="180.34" size="1.778" layer="95">ID_SC</text>
+<text x="327.66" y="177.8" size="1.778" layer="95">MOSI</text>
+<text x="327.66" y="175.26" size="1.778" layer="95">MISO</text>
+<text x="327.66" y="172.72" size="1.778" layer="95">SCLK</text>
+<text x="327.66" y="170.18" size="1.778" layer="95">3.3V</text>
+<text x="358.14" y="190.5" size="1.778" layer="95">5V</text>
+<text x="358.14" y="187.96" size="1.778" layer="95">5V</text>
+<text x="358.14" y="185.42" size="1.778" layer="95">GND</text>
+<text x="358.14" y="182.88" size="1.778" layer="95">TX</text>
+<text x="358.14" y="180.34" size="1.778" layer="95">RX</text>
+<text x="358.14" y="177.8" size="1.778" layer="95">GND</text>
+<text x="358.14" y="170.18" size="1.778" layer="95">GND</text>
+<text x="358.14" y="175.26" size="1.778" layer="95">CE0</text>
+<text x="358.14" y="172.72" size="1.778" layer="95">CE1</text>
+<text x="327.66" y="213.36" size="1.778" layer="95">SDA</text>
+<text x="327.66" y="210.82" size="1.778" layer="95">SCL</text>
+<text x="327.66" y="205.74" size="1.778" layer="95">GND</text>
+<text x="358.14" y="210.82" size="1.778" layer="95">GND</text>
+<text x="358.14" y="215.9" size="1.778" layer="95">5V</text>
+<text x="358.14" y="213.36" size="1.778" layer="95">5V</text>
+<text x="294.64" y="119.38" size="1.778" layer="95">PIR_OUT</text>
+<text x="299.72" y="114.3" size="1.778" layer="95">GND</text>
+<text x="299.72" y="116.84" size="1.778" layer="95">VCC</text>
 </plain>
 <instances>
@@
 <instance part="K1" gate="3" x="228.6" y="434.34" rot="MR180"/>
 <instance part="D2" gate="1" x="513.08" y="220.98" rot="R270"/>
-<instance part="SW1" gate="G$1" x="271.78" y="106.68" rot="MR270"/>
-<instance part="SV15" gate="G$1" x="297.18" y="93.98" rot="R180"/>
-<instance part="SV16" gate="G$1" x="307.34" y="93.98" rot="MR180"/>
+<instance part="SW1" gate="G$1" x="269.24" y="106.68" rot="MR270"/>
+<instance part="SV15" gate="G$1" x="294.64" y="93.98" rot="R180"/>
+<instance part="SV16" gate="G$1" x="309.88" y="93.98" rot="MR180"/>
 <instance part="ULN1" gate="G$1" x="502.92" y="172.72" rot="R90"/>
 <instance part="D1" gate="G$1" x="454.66" y="381" rot="MR90"/>
@@
 <instance part="J9" gate="G$1" x="66.04" y="373.38" rot="R180"/>
 <instance part="J10" gate="G$1" x="495.3" y="360.68" rot="MR90"/>
+<instance part="J11" gate="J$1" x="309.88" y="116.84"/>
 </instances>
 <busses>
@@
 <segment>
 <pinref part="SV16" gate="G$1" pin="2"/>
-<wire x1="314.96" y1="96.52" x2="330.2" y2="96.52" width="0.1524" layer="91"/>
+<wire x1="317.5" y1="96.52" x2="330.2" y2="96.52" width="0.1524" layer="91"/>
 <wire x1="330.2" y1="96.52" x2="330.2" y2="63.5" width="0.1524" layer="91"/>
 <pinref part="GND1" gate="1" pin="GND"/>
@@
 <wire x1="320.04" y1="63.5" x2="330.2" y2="63.5" width="0.1524" layer="91"/>
 <junction x="330.2" y="63.5"/>
+<pinref part="J11" gate="J$1" pin="1"/>
+<wire x1="317.5" y1="114.3" x2="330.2" y2="114.3" width="0.1524" layer="91"/>
+<wire x1="330.2" y1="114.3" x2="330.2" y2="96.52" width="0.1524" layer="91"/>
+<junction x="330.2" y="96.52"/>
 </segment>
 <segment>
@@
 <segment>
 <pinref part="SW1" gate="G$1" pin="SW-"/>
-<wire x1="276.86" y1="116.84" x2="276.86" y2="119.38" width="0.1524" layer="91"/>
+<wire x1="274.32" y1="116.84" x2="274.32" y2="119.38" width="0.1524" layer="91"/>
 <pinref part="SV15" gate="G$1" pin="3"/>
-<wire x1="289.56" y1="93.98" x2="284.48" y2="93.98" width="0.1524" layer="91"/>
-<wire x1="284.48" y1="93.98" x2="284.48" y2="119.38" width="0.1524" layer="91"/>
-<wire x1="284.48" y1="119.38" x2="276.86" y2="119.38" width="0.1524" layer="91"/>
+<wire x1="287.02" y1="93.98" x2="281.94" y2="93.98" width="0.1524" layer="91"/>
+<wire x1="281.94" y1="93.98" x2="281.94" y2="119.38" width="0.1524" layer="91"/>
+<wire x1="281.94" y1="119.38" x2="274.32" y2="119.38" width="0.1524" layer="91"/>
 </segment>
 </net>
@@
 <segment>
 <pinref part="SV15" gate="G$1" pin="1"/>
-<wire x1="289.56" y1="99.06" x2="289.56" y2="121.92" width="0.1524" layer="91"/>
-<wire x1="289.56" y1="121.92" x2="266.7" y2="121.92" width="0.1524" layer="91"/>
+<wire x1="287.02" y1="99.06" x2="287.02" y2="121.92" width="0.1524" layer="91"/>
+<wire x1="287.02" y1="121.92" x2="264.16" y2="121.92" width="0.1524" layer="91"/>
 <pinref part="SW1" gate="G$1" pin="SW+"/>
-<wire x1="266.7" y1="121.92" x2="266.7" y2="116.84" width="0.1524" layer="91"/>
+<wire x1="264.16" y1="121.92" x2="264.16" y2="116.84" width="0.1524" layer="91"/>
 </segment>
 </net>
@@
 <segment>
 <pinref part="SW1" gate="G$1" pin="C"/>
-<wire x1="271.78" y1="93.98" x2="271.78" y2="96.52" width="0.1524" layer="91"/>
+<wire x1="269.24" y1="93.98" x2="269.24" y2="96.52" width="0.1524" layer="91"/>
 <pinref part="SV15" gate="G$1" pin="2"/>
-<wire x1="289.56" y1="96.52" x2="281.94" y2="96.52" width="0.1524" layer="91"/>
-<wire x1="281.94" y1="96.52" x2="281.94" y2="93.98" width="0.1524" layer="91"/>
-<wire x1="281.94" y1="93.98" x2="271.78" y2="93.98" width="0.1524" layer="91"/>
+<wire x1="287.02" y1="96.52" x2="279.4" y2="96.52" width="0.1524" layer="91"/>
+<wire x1="279.4" y1="96.52" x2="279.4" y2="93.98" width="0.1524" layer="91"/>
+<wire x1="279.4" y1="93.98" x2="269.24" y2="93.98" width="0.1524" layer="91"/>
 </segment>
 </net>
@@
 <pinref part="SW1" gate="G$1" pin="A"/>
 <pinref part="SV15" gate="G$1" pin="4"/>
-<wire x1="289.56" y1="91.44" x2="276.86" y2="91.44" width="0.1524" layer="91"/>
-<wire x1="276.86" y1="91.44" x2="276.86" y2="96.52" width="0.1524" layer="91"/>
+<wire x1="287.02" y1="91.44" x2="274.32" y2="91.44" width="0.1524" layer="91"/>
+<wire x1="274.32" y1="91.44" x2="274.32" y2="96.52" width="0.1524" layer="91"/>
 </segment>
 </net>
@@
 <segment>
 <pinref part="SW1" gate="G$1" pin="B"/>
-<wire x1="266.7" y1="96.52" x2="266.7" y2="88.9" width="0.1524" layer="91"/>
+<wire x1="264.16" y1="96.52" x2="264.16" y2="88.9" width="0.1524" layer="91"/>
 <pinref part="SV15" gate="G$1" pin="5"/>
-<wire x1="289.56" y1="88.9" x2="266.7" y2="88.9" width="0.1524" layer="91"/>
+<wire x1="287.02" y1="88.9" x2="264.16" y2="88.9" width="0.1524" layer="91"/>
 </segment>
 </net>
@@
 <segment>
 <pinref part="SV16" gate="G$1" pin="3"/>
-<wire x1="314.96" y1="93.98" x2="320.04" y2="93.98" width="0.1524" layer="91"/>
+<wire x1="317.5" y1="93.98" x2="320.04" y2="93.98" width="0.1524" layer="91"/>
 <wire x1="320.04" y1="93.98" x2="320.04" y2="83.82" width="0.1524" layer="91"/>
 <pinref part="J1" gate="G$1" pin="GP13"/>
@@
 <pinref part="SV16" gate="G$1" pin="5"/>
 <pinref part="J1" gate="G$1" pin="GP6"/>
-<wire x1="314.96" y1="88.9" x2="378.46" y2="88.9" width="0.1524" layer="91"/>
+<wire x1="317.5" y1="88.9" x2="378.46" y2="88.9" width="0.1524" layer="91"/>
 </segment>
 </net>
@@
 <pinref part="SV16" gate="G$1" pin="4"/>
 <pinref part="J1" gate="G$1" pin="GP5"/>
-<wire x1="314.96" y1="91.44" x2="378.46" y2="91.44" width="0.1524" layer="91"/>
+<wire x1="317.5" y1="91.44" x2="378.46" y2="91.44" width="0.1524" layer="91"/>
 </segment>
 </net>
@@
 </segment>
 </net>
-<net name="GROUND" class="1">
+<net name="5V" class="1">
 <segment>
 <pinref part="SV16" gate="G$1" pin="1"/>
-<wire x1="314.96" y1="99.06" x2="335.28" y2="99.06" width="0.1524" layer="91"/>
+<wire x1="317.5" y1="99.06" x2="335.28" y2="99.06" width="0.1524" layer="91"/>
 <wire x1="335.28" y1="99.06" x2="335.28" y2="53.34" width="0.1524" layer="91"/>
 <pinref part="R8" gate="G$1" pin="1"/>
@@
 <pinref part="SV12" gate="G$1" pin="5"/>
 <wire x1="20.32" y1="370.84" x2="15.24" y2="370.84" width="0.1524" layer="91"/>
+<pinref part="J11" gate="J$1" pin="2"/>
+<wire x1="317.5" y1="116.84" x2="335.28" y2="116.84" width="0.1524" layer="91"/>
+<wire x1="335.28" y1="116.84" x2="335.28" y2="99.06" width="0.1524" layer="91"/>
+<junction x="335.28" y="99.06"/>
 </segment>
 </net>
@@
 </segment>
 </net>
+<net name="N$173" class="0">
+<segment>
+<pinref part="J1" gate="G$1" pin="GP16"/>
+<wire x1="378.46" y1="81.28" x2="350.52" y2="81.28" width="0.1524" layer="91"/>
+<wire x1="350.52" y1="81.28" x2="350.52" y2="119.38" width="0.1524" layer="91"/>
+<pinref part="J11" gate="J$1" pin="3"/>
+<wire x1="350.52" y1="119.38" x2="317.5" y2="119.38" width="0.1524" layer="91"/>
+</segment>
+</net>

Commit message: freecad model updated
Parts:
- J11: device SparkFun-Connectors:M03PTH -> con-amp-quick:M03
- J3: device SparkFun-Connectors:M04PTH -> con-amp-quick:M04
- SV16: device SparkFun-Connectors:M05PTH -> con-amp-quick:M05
Changed lines of the file:
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@@
 <part name="SW1" library="SparkFun-Electromechanical" deviceset="ROTARTY_ENCODER" device=""/>
 <part name="SV15" library="SparkFun-Connectors" deviceset="M05" device="PTH"/>
-<part name="SV16" library="SparkFun-Connectors" deviceset="M05" device="PTH"/>
+<part name="SV16" library="con-amp-quick" deviceset="M05" device=""/>
 <part name="ULN1" library="SparkFun-PowerIC" deviceset="ULN2803" device="DIP"/>
 <part name="D1" library="SparkFun-LED" deviceset="LED-RGB-CA-THRU" device="CLEAR"/>
@@
 <part name="SV17" library="con-lstb" deviceset="MA09-2" device=""/>
 <part name="J2" library="SparkFun-Connectors" deviceset="M05X2" device="PTH"/>
-<part name="J3" library="SparkFun-Connectors" deviceset="M04" device="PTH"/>
+<part name="J3" library="con-amp-quick" deviceset="M04" device=""/>
 <part name="J4" library="SparkFun-Connectors" deviceset="M08" device=""/>
 <part name="J5" library="SparkFun-Connectors" deviceset="M08" device=""/>
@@
 <part name="J9" library="SparkFun-Connectors" deviceset="M08" device=""/>
 <part name="J10" library="SparkFun-Connectors" deviceset="M08" device=""/>
-<part name="J11" library="SparkFun-Connectors" deviceset="M03" device="PTH"/>
+<part name="J11" library="con-amp-quick" deviceset="M03" device=""/>
 </parts>
 <sheets>
@@
 <instance part="J9" gate="G$1" x="66.04" y="373.38" rot="R180"/>
 <instance part="J10" gate="G$1" x="495.3" y="360.68" rot="MR90"/>
-<instance part="J11" gate="J$1" x="309.88" y="116.84"/>
+<instance part="J11" gate="G$1" x="309.88" y="116.84"/>
 </instances>
 <busses>
@@
 <wire x1="320.04" y1="63.5" x2="330.2" y2="63.5" width="0.1524" layer="91"/>
 <junction x="330.2" y="63.5"/>
-<pinref part="J11" gate="J$1" pin="1"/>
+<pinref part="J11" gate="G$1" pin="1"/>
 <wire x1="317.5" y1="114.3" x2="330.2" y2="114.3" width="0.1524" layer="91"/>
 <wire x1="330.2" y1="114.3" x2="330.2" y2="96.52" width="0.1524" layer="91"/>
@@
 <pinref part="SV12" gate="G$1" pin="5"/>
 <wire x1="20.32" y1="370.84" x2="15.24" y2="370.84" width="0.1524" layer="91"/>
-<pinref part="J11" gate="J$1" pin="2"/>
+<pinref part="J11" gate="G$1" pin="2"/>
 <wire x1="317.5" y1="116.84" x2="335.28" y2="116.84" width="0.1524" layer="91"/>
 <wire x1="335.28" y1="116.84" x2="335.28" y2="99.06" width="0.1524" layer="91"/>
@@
 <wire x1="378.46" y1="81.28" x2="350.52" y2="81.28" width="0.1524" layer="91"/>
 <wire x1="350.52" y1="81.28" x2="350.52" y2="119.38" width="0.1524" layer="91"/>
-<pinref part="J11" gate="J$1" pin="3"/>
+<pinref part="J11" gate="G$1" pin="3"/>
 <wire x1="350.52" y1="119.38" x2="317.5" y2="119.38" width="0.1524" layer="91"/>
 </segment>

Commit message: Fixed problem related with the pcb
Parts:
- added C19: 0.47uF 300V, resistor:C-EU275-154X316
- added C20: 0,47uF 300V, resistor:C-EU275-154X316
- added C21, C22: (no value), resistor:CPOL-EUE2.5-5
- added R13, R14: 100k, resistor:R-EU_0309/10
- added R15, R16: 10k, resistor:R-EU_0309/10
- added R17, R18: 470k, resistor:R-EU_0309/10
- added R19, R20: 1k2, resistor:R-EU_0309/10
- added R22: PC16D, piher:PC16D
- added V1: (no value), Tubes:ECC82-P
Connections:
- removed net N$145: J1.3.3V@1, J2.1, SV17.1
- new net N$174: R15.1, R17.2
- new net N$175: R16.1, R18.2
- new net N$176: R15.2, V1A.TG
- new net N$177: C20.1, R13.1, V1A.TA
- new net N$178: C19.1, R14.1, V1B.TA
- new net N$179: R16.2, V1B.TG
- new net N$180: C22.+, C22.-, R20.1, R20.2, V1B.TK
- new net N$181: C21.+, R19.2, V1A.TK
- new net N$182: J11.2, R8.1, SV16.1
- new net N$184: C20.2, R22.1A
- new net N$185: C19.2, R22.2A
- net 5V: no longer J11.2, R8.1, SV16.1
- net GND: now also C21.-, R17.1, R18.1, R19.1, R22.1E, R22.2E
- net N$130: now also J1.3.3V@1, J2.1, SV17.1
